File: axiom_core/base_module.kicad_sch (KiCad schematic)
At the start: 1 part, among them J4 DF40C-20DP-0.4V_51_

Commit message: upload
Parts:
- removed J4: DF40C-20DP-0.4V_51_, DF40C-20DP-0.4V_51_:HRS_DF40C-20DP-0.4V_51_, symbol DF40C-20DP-0.4V_51_:DF40C-20DP-0.4V_51_
- added J7: DF40C-20DP-0.4V_51_, Connector_Hirose_DF40:Hirose_DF40C-20DP-0.4V_2x10-1MP_P0.4mm, symbol DF40C-20DP-0.4V_51_:DF40C-20DP-0.4V_51_
Connections:
- net +3V3: now also J7.3, J7.4
- net +5V: now also J7.5, J7.6
- net GND: now also J7.1, J7.17, J7.18, J7.2, J7.7, J7.8
- net GPIO: now also J7.16
- net IRQ: now also J7.15
- net MOD_SCL: now also J7.14
- net MOD_SDA: now also J7.13
- net SPI_CS: now also J7.12
- net SPI_MISO: now also J7.10
- net SPI_MOSI: now also J7.9
- net SPI_SCK: now also J7.11
