File: axiom_core/nrf.kicad_sch (KiCad schematic)
At the start: 20 parts, among them U6 nRF24L01P, U7 RFX2401C, Y3 XL7EL89COI-111YLC-16M

Commit message: upload
Parts:
- C19: renamed from C16; footprint (none) -> Capacitor_SMD:C_0402_1005Metric
- C20: renamed from C23; footprint (none) -> Capacitor_SMD:C_0402_1005Metric
- C21: renamed from C24; footprint (none) -> Capacitor_SMD:C_0402_1005Metric
- C22: renamed from C20; footprint (none) -> Capacitor_SMD:C_0402_1005Metric
- C23: renamed from C19; footprint (none) -> Capacitor_SMD:C_0402_1005Metric
- C24: renamed from C18; footprint (none) -> Capacitor_SMD:C_0402_1005Metric
- C25: renamed from C17; footprint (none) -> Capacitor_SMD:C_0402_1005Metric
- C26: renamed from C21; footprint (none) -> Capacitor_SMD:C_0402_1005Metric
- C27: renamed from C22; footprint (none) -> Capacitor_SMD:C_0402_1005Metric
- C28: renamed from C25; footprint (none) -> Capacitor_SMD:C_0402_1005Metric
- L2: renamed from L3; footprint (none) -> Inductor_SMD:L_0402_1005Metric
- L3: renamed from L2; footprint (none) -> Inductor_SMD:L_0402_1005Metric
- L4: footprint (none) -> Inductor_SMD:L_0402_1005Metric
- R13: renamed from R8; footprint (none) -> Resistor_SMD:R_0402_1005Metric
- R14: renamed from R9; footprint (none) -> Resistor_SMD:R_0402_1005Metric
- R15: renamed from R10; footprint (none) -> Resistor_SMD:R_0402_1005Metric
- R16: renamed from R11; footprint (none) -> Resistor_SMD:R_0402_1005Metric
- U9: renamed from U7; footprint RFX2401C:QFN50P300X300X60-17N -> misclib:RFX2401C
- Y3: footprint (none) -> Crystal:Crystal_SMD_3225-4Pin_3.2x2.5mm
- renumbered U6 to U8
