File: axiom_core/rf_module.kicad_sch (KiCad schematic)
At the start: 1 part, among them J5 DF40C-20DP-0.4V_51_

Commit message: upload
Parts:
- J9: renamed from J5; footprint DF40C-20DP-0.4V_51_:HRS_DF40C-20DP-0.4V_51_ -> Connector_Hirose_DF40:Hirose_DF40C-20DP-0.4V_2x10-1MP_P0.4mm
Changed lines of the file:
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@@
 		(dnp no)
 		(fields_autoplaced yes)
-		(property "Reference" "J5"
+		(property "Reference" "J9"
 			(at 147.32 74.93 0)
 			(effects
@@
 			)
 		)
-		(property "Footprint" "DF40C-20DP-0.4V_51_:HRS_DF40C-20DP-0.4V_51_"
+		(property "Footprint" "Connector_Hirose_DF40:Hirose_DF40C-20DP-0.4V_2x10-1MP_P0.4mm"
 			(at 147.32 95.25 0)
 			(effects
@@
 			(project "axiom_core"
 				(path "/71d130ab-f2cb-4bba-8902-75557e00a435/f69ec053-b227-4d5c-8e1c-e6bfd2f76e61"
-					(reference "J5")
+					(reference "J9")
 					(unit 1)
 				)
@@
 		(dnp no)
 		(fields_autoplaced yes)
-		(property "Reference" "#PWR056"
+		(property "Reference" "#PWR067"
 			(at 116.84 106.68 0)
 			(effects
@@
 			(project "axiom_core"
 				(path "/71d130ab-f2cb-4bba-8902-75557e00a435/f69ec053-b227-4d5c-8e1c-e6bfd2f76e61"
-					(reference "#PWR056")
+					(reference "#PWR067")
 					(unit 1)
 				)
@@
 		(dnp no)
 		(fields_autoplaced yes)
-		(property "Reference" "#PWR060"
+		(property "Reference" "#PWR071"
 			(at 173.99 104.14 0)
 			(effects
@@
 			(project "axiom_core"
 				(path "/71d130ab-f2cb-4bba-8902-75557e00a435/f69ec053-b227-4d5c-8e1c-e6bfd2f76e61"
-					(reference "#PWR060")
+					(reference "#PWR071")
 					(unit 1)
 				)
@@
 		(dnp no)
 		(fields_autoplaced yes)
-		(property "Reference" "#PWR058"
+		(property "Reference" "#PWR069"
 			(at 134.62 111.76 0)
 			(effects
@@
 			(project "axiom_core"
 				(path "/71d130ab-f2cb-4bba-8902-75557e00a435/f69ec053-b227-4d5c-8e1c-e6bfd2f76e61"
-					(reference "#PWR058")
+					(reference "#PWR069")
 					(unit 1)
 				)
@@
 		(dnp no)
 		(fields_autoplaced yes)
-		(property "Reference" "#PWR061"
+		(property "Reference" "#PWR072"
 			(at 177.8 106.68 0)
 			(effects
@@
 			(project "axiom_core"
 				(path "/71d130ab-f2cb-4bba-8902-75557e00a435/f69ec053-b227-4d5c-8e1c-e6bfd2f76e61"
-					(reference "#PWR061")
+					(reference "#PWR072")
 					(unit 1)
 				)
@@
 		(dnp no)
 		(fields_autoplaced yes)
-		(property "Reference" "#PWR057"
+		(property "Reference" "#PWR068"
 			(at 120.65 104.14 0)
 			(effects
@@
 			(project "axiom_core"
 				(path "/71d130ab-f2cb-4bba-8902-75557e00a435/f69ec053-b227-4d5c-8e1c-e6bfd2f76e61"
-					(reference "#PWR057")
+					(reference "#PWR068")
 					(unit 1)
 				)
@@
 		(dnp no)
 		(fields_autoplaced yes)
-		(property "Reference" "#PWR059"
+		(property "Reference" "#PWR070"
 			(at 160.02 111.76 0)
 			(effects
@@
 			(project "axiom_core"
 				(path "/71d130ab-f2cb-4bba-8902-75557e00a435/f69ec053-b227-4d5c-8e1c-e6bfd2f76e61"
-					(reference "#PWR059")
-					(unit 1)
-				)
+					(reference "#PWR070")
+					(unit 1)
+				)
