File: axiom_core/ui.kicad_sch (KiCad schematic)
At the start: 9 parts, among them SW3 SEL, SW4 BCK, SW5 LEFT, SW6 UP, SW7 RIGHT, SW8 DOWN, U11 MCP23008-xML

Commit message: upload
Parts:
- C39: renamed from C36; footprint (none) -> Capacitor_SMD:C_0402_1005Metric
- R21: renamed from R16; footprint (none) -> Resistor_SMD:R_0402_1005Metric
- SW4: renamed from SW5; footprint (none) -> Button_Switch_SMD:SW_SPST_B3U-1000P
- SW5: renamed from SW6; footprint (none) -> Button_Switch_SMD:SW_SPST_B3U-1000P
- SW6: renamed from SW8; footprint (none) -> Button_Switch_SMD:SW_SPST_B3U-1000P
- SW7: footprint (none) -> Button_Switch_SMD:SW_SPST_B3U-1000P
- SW8: renamed from SW3; footprint (none) -> Button_Switch_SMD:SW_SPST_B3U-1000P
- SW9: renamed from SW4; footprint (none) -> Button_Switch_SMD:SW_SPST_B3U-1000P
- renumbered U11 to U12
Changed lines of the file:
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@@
 		(dnp no)
 		(fields_autoplaced yes)
-		(property "Reference" "#PWR036"
+		(property "Reference" "#PWR046"
 			(at 33.02 113.03 0)
 			(effects
@@
 			(project "axiom_core"
 				(path "/71d130ab-f2cb-4bba-8902-75557e00a435/51b9f496-ea5b-4994-8444-d894c16bfa05"
-					(reference "#PWR036")
+					(reference "#PWR046")
 					(unit 1)
 				)
@@
 		(dnp no)
 		(fields_autoplaced yes)
-		(property "Reference" "#PWR037"
+		(property "Reference" "#PWR045"
 			(at 27.94 107.95 0)
 			(effects
@@
 			(project "axiom_core"
 				(path "/71d130ab-f2cb-4bba-8902-75557e00a435/51b9f496-ea5b-4994-8444-d894c16bfa05"
-					(reference "#PWR037")
+					(reference "#PWR045")
 					(unit 1)
 				)
@@
 			)
 		)
-		(property "Footprint" ""
+		(property "Footprint" "Button_Switch_SMD:SW_SPST_B3U-1000P"
 			(at 157.48 115.57 0)
 			(effects
@@
 		(dnp no)
 		(fields_autoplaced yes)
-		(property "Reference" "#PWR043"
+		(property "Reference" "#PWR050"
 			(at 139.7 111.76 0)
 			(effects
@@
 			(project "axiom_core"
 				(path "/71d130ab-f2cb-4bba-8902-75557e00a435/51b9f496-ea5b-4994-8444-d894c16bfa05"
-					(reference "#PWR043")
+					(reference "#PWR050")
 					(unit 1)
 				)
@@
 		(dnp no)
 		(fields_autoplaced yes)
-		(property "Reference" "SW8"
+		(property "Reference" "SW6"
 			(at 143.51 125.7299 90)
 			(effects
@@
 			)
 		)
-		(property "Footprint" ""
+		(property "Footprint" "Button_Switch_SMD:SW_SPST_B3U-1000P"
 			(at 144.78 127 0)
 			(effects
@@
 			(project "axiom_core"
 				(path "/71d130ab-f2cb-4bba-8902-75557e00a435/51b9f496-ea5b-4994-8444-d894c16bfa05"
-					(reference "SW8")
+					(reference "SW6")
 					(unit 1)
 				)
@@
 		(dnp no)
 		(fields_autoplaced yes)
-		(property "Reference" "SW3"
+		(property "Reference" "SW8"
 			(at 185.42 114.2999 90)
 			(effects
@@
 			)
 		)
-		(property "Footprint" ""
+		(property "Footprint" "Button_Switch_SMD:SW_SPST_B3U-1000P"
 			(at 186.69 115.57 0)
 			(effects
@@
 			(project ""
 				(path "/71d130ab-f2cb-4bba-8902-75557e00a435/51b9f496-ea5b-4994-8444-d894c16bfa05"
-					(reference "SW3")
+					(reference "SW8")
 					(unit 1)
 				)
@@
 		(dnp no)
 		(fields_autoplaced yes)
-		(property "Reference" "U11"
+		(property "Reference" "U12"
 			(at 55.4833 101.6 0)
 			(effects
@@
 			(project "axiom_core"
 				(path "/71d130ab-f2cb-4bba-8902-75557e00a435/51b9f496-ea5b-4994-8444-d894c16bfa05"
-					(reference "U11")
+					(reference "U12")
 					(unit 1)
 				)
@@
 		(dnp no)
 		(fields_autoplaced yes)
-		(property "Reference" "#PWR034"
+		(property "Reference" "#PWR048"
 			(at 53.34 140.97 0)
 			(effects
@@
 			(project ""
 				(path "/71d130ab-f2cb-4bba-8902-75557e00a435/51b9f496-ea5b-4994-8444-d894c16bfa05"
-					(reference "#PWR034")
+					(reference "#PWR048")
 					(unit 1)
 				)
@@
 		(on_board yes)
 		(dnp no)
-		(property "Reference" "R16"
+		(property "Reference" "R21"
 			(at 38.354 104.14 90)
 			(effects
@@
 			)
 		)
-		(property "Footprint" ""
+		(property "Footprint" "Resistor_SMD:R_0402_1005Metric"
 			(at 36.83 110.998 90)
 			(effects
@@
 			(project ""
 				(path "/71d130ab-f2cb-4bba-8902-75557e00a435/51b9f496-ea5b-4994-8444-d894c16bfa05"
-					(reference "R16")
+					(reference "R21")
 					(unit 1)
 				)
@@
 		(dnp no)
 		(fields_autoplaced yes)
-		(property "Reference" "#PWR041"
+		(property "Reference" "#PWR053"
 			(at 181.61 127 0)
 			(effects
@@
 			(project "axiom_core"
 				(path "/71d130ab-f2cb-4bba-8902-75557e00a435/51b9f496-ea5b-4994-8444-d894c16bfa05"
-					(reference "#PWR041")
+					(reference "#PWR053")
 					(unit 1)
 				)
@@
 		(on_board yes)
 		(dnp no)
-		(property "Reference" "C36"
+		(property "Reference" "C39"
 			(at 57.404 97.028 90)
 			(effects
@@
 			)
 		)
-		(property "Footprint" ""
+		(property "Footprint" "Capacitor_SMD:C_0402_1005Metric"
 			(at 50.8 101.6 0)
 			(effects
@@
 			(project ""
 				(path "/71d130ab-f2cb-4bba-8902-75557e00a435/51b9f496-ea5b-4994-8444-d894c16bfa05"
-					(reference "C36")
+					(reference "C39")
 					(unit 1)
 				)
@@
 		(dnp no)
 		(fields_autoplaced yes)
-		(property "Reference" "SW4"
+		(property "Reference" "SW9"
 			(at 208.28 114.2999 90)
 			(effects
@@
 			)
 		)
-		(property "Footprint" ""
+		(property "Footprint" "Button_Switch_SMD:SW_SPST_B3U-1000P"
 			(at 209.55 115.57 0)
 			(effects
@@
 			(project "axiom_core"
 				(path "/71d130ab-f2cb-4bba-8902-75557e00a435/51b9f496-ea5b-4994-8444-d894c16bfa05"
-					(reference "SW4")
+					(reference "SW9")
 					(unit 1)
 				)
@@
 		(dnp no)
 		(fields_autoplaced yes)
-		(property "Reference" "#PWR038"
+		(property "Reference" "#PWR051"
 			(at 139.7 138.43 0)
 			(effects
@@
 			(project "axiom_core"
 				(path "/71d130ab-f2cb-4bba-8902-75557e00a435/51b9f496-ea5b-4994-8444-d894c16bfa05"
-					(reference "#PWR038")
+					(reference "#PWR051")
 					(unit 1)
 				)
@@
 		(dnp no)
 		(fields_autoplaced yes)
-		(property "Reference" "#PWR042"
+		(property "Reference" "#PWR054"
 			(at 204.47 127 0)
 			(effects
@@
 			(project "axiom_core"
 				(path "/71d130ab-f2cb-4bba-8902-75557e00a435/51b9f496-ea5b-4994-8444-d894c16bfa05"
-					(reference "#PWR042")
+					(reference "#PWR054")
 					(unit 1)
 				)
@@
 		(dnp no)
 		(fields_autoplaced yes)
-		(property "Reference" "SW6"
+		(property "Reference" "SW5"
 			(at 143.51 99.0599 90)
 			(effects
@@
 			)
 		)
-		(property "Footprint" ""
+		(property "Footprint" "Button_Switch_SMD:SW_SPST_B3U-1000P"
 			(at 144.78 100.33 0)
 			(effects
@@
 			(project "axiom_core"
 				(path "/71d130ab-f2cb-4bba-8902-75557e00a435/51b9f496-ea5b-4994-8444-d894c16bfa05"
-					(reference "SW6")
+					(reference "SW5")
 					(unit 1)
 				)
@@
 		(dnp no)
 		(fields_autoplaced yes)
-		(property "Reference" "#PWR040"
+		(property "Reference" "#PWR052"
 			(at 152.4 127 0)
 			(effects
@@
 			(project "axiom_core"
 				(path "/71d130ab-f2cb-4bba-8902-75557e00a435/51b9f496-ea5b-4994-8444-d894c16bfa05"
-					(reference "#PWR040")
+					(reference "#PWR052")
 					(unit 1)
 				)
@@
 		(dnp no)
 		(fields_autoplaced yes)
-		(property "Reference" "#PWR035"
+		(property "Reference" "#PWR047"
 			(at 53.34 102.87 0)
 			(effects
@@
 			(project ""
 				(path "/71d130ab-f2cb-4bba-8902-75557e00a435/51b9f496-ea5b-4994-8444-d894c16bfa05"
-					(reference "#PWR035")
+					(reference "#PWR047")
 					(unit 1)
 				)
@@
 		(dnp no)
 		(fields_autoplaced yes)
-		(property "Reference" "SW5"
+		(property "Reference" "SW4"
 			(at 128.27 113.0299 90)
 			(effects
@@
 			)
 		)
-		(property "Footprint" ""
+		(property "Footprint" "Button_Switch_SMD:SW_SPST_B3U-1000P"
 			(at 129.54 114.3 0)
 			(effects
@@
 			(project "axiom_core"
 				(path "/71d130ab-f2cb-4bba-8902-75557e00a435/51b9f496-ea5b-4994-8444-d894c16bfa05"
-					(reference "SW5")
+					(reference "SW4")
 					(unit 1)
 				)
@@
 		(dnp no)
 		(fields_autoplaced yes)
-		(property "Reference" "#PWR039"
+		(property "Reference" "#PWR049"
 			(at 124.46 125.73 0)
 			(effects
@@
 			(project "axiom_core"
 				(path "/71d130ab-f2cb-4bba-8902-75557e00a435/51b9f496-ea5b-4994-8444-d894c16bfa05"
-					(reference "#PWR039")
-					(unit 1)
-				)
+					(reference "#PWR049")
+					(unit 1)
+				)
