File: axiom_core/mcu.kicad_sch (KiCad schematic)
At the start: 30 parts, among them SW1 BOOT, SW2 RST, U12 PCA9536D, U3 ESP32-S3, U4 W25Q128JVSIQ, Y1 EPSON Q13FC13500004, Y2 TROQ RG40000421

Commit message: upload
Parts:
- C10: renamed from C2; footprint (none) -> Capacitor_SMD:C_0402_1005Metric
- C11: renamed from C3; footprint (none) -> Capacitor_SMD:C_0402_1005Metric
- C12: renamed from C4; footprint (none) -> Capacitor_SMD:C_0402_1005Metric
- C13: renamed from C5; footprint (none) -> Capacitor_SMD:C_0402_1005Metric
- C14: renamed from C6; footprint (none) -> Capacitor_SMD:C_0402_1005Metric
- C15: renamed from C9; footprint (none) -> Capacitor_SMD:C_0402_1005Metric
- C16: renamed from C10; footprint (none) -> Capacitor_SMD:C_0402_1005Metric
- C17: renamed from C8; footprint (none) -> Capacitor_SMD:C_0402_1005Metric
- C18: renamed from C15; footprint (none) -> Capacitor_SMD:C_0402_1005Metric
- C3: renamed from C37; footprint (none) -> Capacitor_SMD:C_0402_1005Metric
- C4: renamed from C14; footprint (none) -> Capacitor_SMD:C_0402_1005Metric
- C5: renamed from C13; footprint (none) -> Capacitor_SMD:C_0402_1005Metric
- C6: renamed from C12; footprint (none) -> Capacitor_SMD:C_0402_1005Metric
- C7: renamed from C11; footprint (none) -> Capacitor_SMD:C_0402_1005Metric
- C8: renamed from C7; footprint (none) -> Capacitor_SMD:C_0402_1005Metric
- C9: renamed from C1; footprint (none) -> Capacitor_SMD:C_0402_1005Metric
- L1: footprint (none) -> Inductor_SMD:L_0402_1005Metric
- R10: renamed from R20; footprint (none) -> Resistor_SMD:R_0402_1005Metric
- R11: renamed from R5; footprint (none) -> Resistor_SMD:R_0402_1005Metric
- R12: renamed from R4; footprint (none) -> Resistor_SMD:R_0402_1005Metric
- R9: renamed from R19; footprint (none) -> Resistor_SMD:R_0402_1005Metric
- SW2: renamed from SW1; footprint (none) -> Button_Switch_SMD:SW_SPST_B3U-1000P
- SW3: renamed from SW2; footprint (none) -> Button_Switch_SMD:SW_SPST_B3U-1000P
- TP1, TP2: footprint (none) -> TestPoint:TestPoint_Pad_D1.0mm
- U5: renamed from U12; footprint PCA9536D:SOIC127P599X175-8N -> misclib:SOIC127P599X175-8N
- Y1: renamed from Y2; footprint (none) -> Crystal:Crystal_SMD_5032-2Pin_5.0x3.2mm
- Y2: renamed from Y1; footprint (none) -> Crystal:Crystal_SMD_3225-4Pin_3.2x2.5mm
- renumbered U3 to U6, U4 to U7

Commit message: upload
Changed lines of the file:
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@@
 		(lib_id "Device:R_Small")
 		(at 158.75 147.32 0)
+		(mirror y)
 		(unit 1)
 		(exclude_from_sim no)
@@
 		(on_board yes)
 		(dnp no)
-		(fields_autoplaced yes)
 		(property "Reference" "R12"
-			(at 161.29 146.0499 0)
+			(at 156.21 146.0499 0)
 			(effects
 				(font
@@
 		)
 		(property "Value" "10k"
-			(at 161.29 148.5899 0)
+			(at 156.21 148.5899 0)
 			(effects
 				(font
