File: axiom_core/power_sheet.kicad_sch (KiCad schematic)
At the start: 9 parts, among them J1 USB_C_Receptacle_USB2.0_14P, U1 TPS2113APW, U2 AMS1117-3.3, U5 USBLC6-2P6

Commit message: upload
Parts:
- added C38: 22uF, symbol Device:C
- added C39: 10uF, symbol Device:C
- added SW9: PWR, symbol Switch:SW_SPST
Connections:
- net +3V3: now also SW9.2 (B); no longer U2.2 (VO)
- net +5V: now also C39.1
- net at U1.5 (GND), U2.1 (GND): now also C38.2, C39.2
- new net: C38.1, SW9.1 (A), U2.2 (VO)
Other:
- moved on the sheet: J1, R1, R2, R3, R6, R7, U1, U2, U5

Commit message: upload
Parts:
- C1: renamed from C39; footprint (none) -> Capacitor_SMD:C_0402_1005Metric
- C2: renamed from C38; footprint (none) -> Capacitor_SMD:C_0402_1005Metric
- J6: renamed from J1; footprint (none) -> Connector_USB:USB_C_Receptacle_HRO_TYPE-C-31-M-12
- R4: renamed from R2; footprint (none) -> Resistor_SMD:R_0402_1005Metric
- R5: renamed from R3; footprint (none) -> Resistor_SMD:R_0402_1005Metric
- R6, R7: footprint (none) -> Resistor_SMD:R_0402_1005Metric
- R8: renamed from R1; footprint (none) -> Resistor_SMD:R_0402_1005Metric
- SW1: renamed from SW9; footprint (none) -> Button_Switch_SMD:SW_SPST_B3U-1000P
- renumbered U5 to U2, U1 to U3, U2 to U4
Changed lines of the file:
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@@
 		(dnp no)
 		(fields_autoplaced yes)
-		(property "Reference" "#PWR031"
+		(property "Reference" "#PWR012"
 			(at 55.88 119.38 0)
 			(effects
@@
 			(project "axiom_core"
 				(path "/71d130ab-f2cb-4bba-8902-75557e00a435/c9714ede-cda4-4a3e-a365-b1de95545e37"
-					(reference "#PWR031")
+					(reference "#PWR012")
 					(unit 1)
 				)
@@
 		(dnp no)
 		(fields_autoplaced yes)
-		(property "Reference" "U1"
+		(property "Reference" "U3"
 			(at 124.46 59.69 0)
 			(effects
@@
 			(project ""
 				(path "/71d130ab-f2cb-4bba-8902-75557e00a435/c9714ede-cda4-4a3e-a365-b1de95545e37"
-					(reference "U1")
+					(reference "U3")
 					(unit 1)
 				)
@@
 		(dnp no)
 		(fields_autoplaced yes)
-		(property "Reference" "#PWR016"
+		(property "Reference" "#PWR014"
 			(at 161.29 76.2 0)
 			(effects
@@
 			(project ""
 				(path "/71d130ab-f2cb-4bba-8902-75557e00a435/c9714ede-cda4-4a3e-a365-b1de95545e37"
-					(reference "#PWR016")
+					(reference "#PWR014")
 					(unit 1)
 				)
@@
 		(dnp no)
 		(fields_autoplaced yes)
-		(property "Reference" "SW9"
+		(property "Reference" "SW1"
 			(at 191.77 63.4999 90)
 			(effects
@@
 			)
 		)
-		(property "Footprint" ""
+		(property "Footprint" "Button_Switch_SMD:SW_SPST_B3U-1000P"
 			(at 190.5 64.77 0)
 			(effects
@@
 			(project ""
 				(path "/71d130ab-f2cb-4bba-8902-75557e00a435/c9714ede-cda4-4a3e-a365-b1de95545e37"
-					(reference "SW9")
+					(reference "SW1")
 					(unit 1)
 				)
@@
 		(on_board yes)
 		(dnp no)
-		(property "Reference" "U5"
+		(property "Reference" "U2"
 			(at 89.4781 77.47 0)
 			(effects
@@
 			(project ""
 				(path "/71d130ab-f2cb-4bba-8902-75557e00a435/c9714ede-cda4-4a3e-a365-b1de95545e37"
-					(reference "U5")
+					(reference "U2")
 					(unit 1)
 				)
@@
 		(dnp no)
 		(fields_autoplaced yes)
-		(property "Reference" "R1"
+		(property "Reference" "R8"
 			(at 99.06 69.85 90)
 			(effects
@@
 			)
 		)
-		(property "Footprint" ""
+		(property "Footprint" "Resistor_SMD:R_0402_1005Metric"
 			(at 99.06 74.93 0)
 			(effects
@@
 			(project ""
 				(path "/71d130ab-f2cb-4bba-8902-75557e00a435/c9714ede-cda4-4a3e-a365-b1de95545e37"
-					(reference "R1")
+					(reference "R8")
 					(unit 1)
 				)
@@
 		(dnp no)
 		(fields_autoplaced yes)
-		(property "Reference" "C38"
+		(property "Reference" "C2"
 			(at 190.5 74.9299 0)
 			(effects
@@
 			)
 		)
-		(property "Footprint" ""
+		(property "Footprint" "Capacitor_SMD:C_0402_1005Metric"
 			(at 187.6552 80.01 0)
 			(effects
@@
 			(project ""
 				(path "/71d130ab-f2cb-4bba-8902-75557e00a435/c9714ede-cda4-4a3e-a365-b1de95545e37"
-					(reference "C38")
+					(reference "C2")
 					(unit 1)
 				)
@@
 		(dnp no)
 		(fields_autoplaced yes)
-		(property "Reference" "J1"
+		(property "Reference" "J6"
 			(at 55.88 62.23 0)
 			(effects
@@
 			)
 		)
-		(property "Footprint" ""
+		(property "Footprint" "Connector_USB:USB_C_Receptacle_HRO_TYPE-C-31-M-12"
 			(at 59.69 85.09 0)
 			(effects
@@
 			(project ""
 				(path "/71d130ab-f2cb-4bba-8902-75557e00a435/c9714ede-cda4-4a3e-a365-b1de95545e37"
-					(reference "J1")
+					(reference "J6")
 					(unit 1)
 				)
@@
 		(dnp no)
 		(fields_autoplaced yes)
-		(property "Reference" "U2"
+		(property "Reference" "U4"
 			(at 175.26 66.04 0)
 			(effects
@@
 			(project ""
 				(path "/71d130ab-f2cb-4bba-8902-75557e00a435/c9714ede-cda4-4a3e-a365-b1de95545e37"
-					(reference "U2")
+					(reference "U4")
 					(unit 1)
 				)
@@
 		(on_board yes)
 		(dnp no)
-		(property "Reference" "R3"
+		(property "Reference" "R5"
 			(at 73.66 76.454 90)
 			(effects
@@
 			)
 		)
-		(property "Footprint" ""
+		(property "Footprint" "Resistor_SMD:R_0402_1005Metric"
 			(at 73.66 77.47 0)
 			(effects
@@
 			(project "axiom_core"
 				(path "/71d130ab-f2cb-4bba-8902-75557e00a435/c9714ede-cda4-4a3e-a365-b1de95545e37"
-					(reference "R3")
+					(reference "R5")
 					(unit 1)
 				)
@@
 			)
 		)
-		(property "Footprint" ""
+		(property "Footprint" "Resistor_SMD:R_0402_1005Metric"
 			(at 78.74 87.63 0)
 			(effects
@@
 		(on_board yes)
 		(dnp no)
-		(property "Reference" "R2"
+		(property "Reference" "R4"
 			(at 73.66 72.136 90)
 			(effects
@@
 			)
 		)
-		(property "Footprint" ""
+		(property "Footprint" "Resistor_SMD:R_0402_1005Metric"
 			(at 73.66 74.93 0)
 			(effects
@@
 			(project "axiom_core"
 				(path "/71d130ab-f2cb-4bba-8902-75557e00a435/c9714ede-cda4-4a3e-a365-b1de95545e37"
-					(reference "R2")
+					(reference "R4")
 					(unit 1)
 				)
@@
 			)
 		)
-		(property "Footprint" ""
+		(property "Footprint" "Resistor_SMD:R_0402_1005Metric"
 			(at 78.74 85.09 0)
 			(effects
@@
 		(dnp no)
 		(fields_autoplaced yes)
-		(property "Reference" "#PWR014"
+		(property "Reference" "#PWR013"
 			(at 92.71 95.25 0)
 			(effects
@@
 			(project ""
 				(path "/71d130ab-f2cb-4bba-8902-75557e00a435/c9714ede-cda4-4a3e-a365-b1de95545e37"
-					(reference "#PWR014")
+					(reference "#PWR013")
 					(unit 1)
 				)
@@
 		(dnp no)
 		(fields_autoplaced yes)
-		(property "Reference" "C39"
+		(property "Reference" "C1"
 			(at 160.02 74.9299 0)
 			(effects
@@
 			)
 		)
-		(property "Footprint" ""
+		(property "Footprint" "Capacitor_SMD:C_0402_1005Metric"
 			(at 157.1752 80.01 0)
 			(effects
@@
 			(project "axiom_core"
 				(path "/71d130ab-f2cb-4bba-8902-75557e00a435/c9714ede-cda4-4a3e-a365-b1de95545e37"
-					(reference "C39")
-					(unit 1)
-				)
+					(reference "C1")
+					(unit 1)
+				)

Commit message: upload
Connections:
- net GND: now also C1.2, C2.2, R4.2, R5.2, R8.1, U3.2 (~{EN}), U3.5 (GND), U4.1 (GND)
Changed lines of the file:
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@@
+	)
+	(junction
+		(at 81.28 73.66)
+		(diameter 0)
+		(color 0 0 0 0)
 	)
 	(junction
@@
 	(wire
 		(pts
-			(xy 77.47 73.66) (xy 95.25 73.66)
+			(xy 77.47 73.66) (xy 81.28 73.66)
 		)
 		(stroke
@@
 		(pts
 			(xy 189.23 72.39) (xy 190.5 71.12)
+		)
+		(stroke
+			(width 0)
+			(type default)
+		)
+	)
+	(wire
+		(pts
+			(xy 81.28 73.66) (xy 95.25 73.66)
 		)
 		(stroke
@@
 					(unit 1)
 				)
+			)
+		)
+	)
+	(symbol
+		(lib_id "power:GND")
+		(at 163.83 87.63 0)
+		(unit 1)
+		(exclude_from_sim no)
+		(in_bom yes)
+		(on_board yes)
+		(dnp no)
+		(fields_autoplaced yes)
+		(property "Reference" "#PWR074"
+			(at 163.83 93.98 0)
+			(effects
+				(font
+					(size 1.27 1.27)
+				)
+				(hide yes)
+			)
+		)
+		(property "Value" "GND"
+			(at 163.83 92.71 0)
+			(effects
+				(font
+					(size 1.27 1.27)
+				)
+			)
+		)
+		(property "Footprint" ""
+			(at 163.83 87.63 0)
+			(effects
+				(font
+					(size 1.27 1.27)
+				)
+				(hide yes)
+			)
+		)
+		(property "Datasheet" ""
+			(at 163.83 87.63 0)
+			(effects
+				(font
+					(size 1.27 1.27)
+				)
+				(hide yes)
+			)
+		)
+		(property "Description" "Power symbol creates a global label with name \"GND\" , ground"
+			(at 163.83 87.63 0)
+			(effects
+				(font
+					(size 1.27 1.27)
+				)
+				(hide yes)
+			)
+		)
+		(pin "1"
+		)
+		(instances
+			(project "axiom_core"
+				(path "/71d130ab-f2cb-4bba-8902-75557e00a435/c9714ede-cda4-4a3e-a365-b1de95545e37"
+					(reference "#PWR074")
+					(unit 1)
+				)
+			)
+		)
+	)
+	(symbol
+		(lib_id "power:GND")
+		(at 81.28 73.66 0)
+		(unit 1)
+		(exclude_from_sim no)
+		(in_bom yes)
+		(on_board yes)
+		(dnp no)
+		(fields_autoplaced yes)
+		(property "Reference" "#PWR073"
+			(at 81.28 80.01 0)
+			(effects
+				(font
+					(size 1.27 1.27)
+				)
+				(hide yes)
+			)
+		)
+		(property "Value" "GND"
+			(at 81.28 78.74 0)
+			(effects
+				(font
+					(size 1.27 1.27)
+				)
+			)
+		)
+		(property "Footprint" ""
+			(at 81.28 73.66 0)
+			(effects
+				(font
+					(size 1.27 1.27)
+				)
+				(hide yes)
+			)
+		)
+		(property "Datasheet" ""
+			(at 81.28 73.66 0)
+			(effects
+				(font
+					(size 1.27 1.27)
+				)
+				(hide yes)
+			)
+		)
+		(property "Description" "Power symbol creates a global label with name \"GND\" , ground"
+			(at 81.28 73.66 0)
+			(effects
+				(font
+					(size 1.27 1.27)
+				)
+				(hide yes)
+			)
+		)
+		(pin "1"
+		)
+		(instances
+			(project "axiom_core"
+				(path "/71d130ab-f2cb-4bba-8902-75557e00a435/c9714ede-cda4-4a3e-a365-b1de95545e37"
+					(reference "#PWR073")
+					(unit 1)
+				)
