File: axiom_core/axiom_core.kicad_pcb (KiCad board)
At the start: 2 copper layers, 88.2 x 169.7 mm, 104 parts, among them J6 USB_C_Receptacle_USB2.0_14P, J7 DF40C-20DP-0.4V_51_, J8 DF40C-20DP-0.4V_51_, J9 DF40C-20DP-0.4V_51_, K1 drill_guide, SW1 PWR, SW2 BOOT, SW3 RST, SW4 LEFT, SW5 UP, SW6 DOWN, SW7 RIGHT, SW8 SEL, SW9 BCK, U1 CR2013-MI2120, U10 nRF24L01P, U11 RFX2401C, U12 MCP23008-xML, U2 USBLC6-2P6, U3 TPS2113APW, U4 AMS1117-3.3, U5 PCA9536D, U6 ESP32-S3, U7 W25Q128JVSIQ, U8 nRF24L01P, U9 RFX2401C, Y1 TROQ RG40000421, Y2 EPSON Q13FC13500004, Y3 XL7EL89COI-111YLC-16M, Y4 XL7EL89COI-111YLC-16M

Commit message: upload
Parts:
- removed SW1: PWR, Button_Switch_SMD:SW_SPST_B3U-1000P
- added PWR: SW_Slide_SPDT_Angled_CK_OS102011MA1Q, Button_Switch_THT:SW_Slide_SPDT_Angled_CK_OS102011MA1Q, F.Cu at (133.0, 71.0)
- moved MOD_RF 224.8 mm to (77.8, 31.9), turned to 180 degrees
- moved R21 214.9 mm to (74.5, 160.5)
- moved U12 214.5 mm to (78.5, 160.0)
- moved C39 211.4 mm to (79.5, 156.5), turned to 180 degrees
- moved LEFT 198.8 mm to (88.7, 157.5)
- moved JMOD_0 191.3 mm to (78.3, 130.6)
- moved DOWN 190.5 mm to (95.7, 161.5)
- moved UP 188.9 mm to (95.7, 153.5)
- moved U11 185.4 mm to (114.9, 32.2), turned to 90 degrees
- moved BOOT 184.9 mm to (63.0, 24.0)
- moved C38 184.4 mm to (111.5, 32.5), turned to -90 degrees
- moved RST 184.2 mm to (63.0, 29.5)
- moved RIGHT 180.1 mm to (103.2, 157.5)
- moved JMOD_1 179.7 mm to (78.3, 112.4)
- moved C37 177.7 mm to (116.5, 35.0), turned to 180 degrees
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- renumbered ESP32 to 2.4G, SW9 to BCK, SW2 to BOOT, SW6 to DOWN, SHIELD to J1, J7 to JMOD_0, J8 to JMOD_1, NRF1 to JNRF1, NRF2 to JNRF2, SW4 to LEFT, J9 to MOD_RF, RF1 to RF0, SW7 to RIGHT, SW3 to RST, TP2 to RX, SW8 to SEL, TP1 to TX, SW5 to UP
Connections:
- C1 pad 2: Net-(U3-GND) -> GND
- C2 pad 2: Net-(U3-GND) -> GND
- R4 pad 2: Net-(U3-~{EN}) -> GND
- R5 pad 2: Net-(U3-~{EN}) -> GND
- R8 pad 1: Net-(U3-~{EN}) -> GND
- U1 pad 3: /DISP_CS -> /MCU/LCD_CS
- U3 pad 2: Net-(U3-~{EN}) -> GND
- U3 pad 5: Net-(U3-GND) -> GND
- U4 pad 1: Net-(U3-GND) -> GND
- Y2 pad 3: (no net) -> GND
- Y2 pad 4: (no net) -> GND
Routing:
- net +5V: track 0.00 -> 292.8 mm, vias 0 -> 2
- net +3V3: track 0.00 -> 199.2 mm, vias 0 -> 14
- net GND: track 0.00 -> 198.5 mm, vias 0 -> 112
- net /MAIN_MISO: track 0.00 -> 154.6 mm, vias 0 -> 2
- net /MAIN_MOSI: track 0.00 -> 154.0 mm, vias 0 -> 2
- net /MAIN_SCLK: track 0.00 -> 153.0 mm, vias 0 -> 5
- net /BTN_IRQ: track 0.00 -> 105.3 mm, vias 0 -> 2
- net /MCU/LCD_CS: track 0.00 -> 91.0 mm, vias 0 -> 2
- net /GPIO0: track 0.00 -> 80.9 mm, vias 0 -> 2
- net /button_manager/SEL: track 0.00 -> 68.0 mm
- net Net-(U3-IN1): track 0.00 -> 61.3 mm, vias 0 -> 3
- net /NRF2_RXEN: track 0.00 -> 52.8 mm, vias 0 -> 2
- net /NRF2_TXEN: track 0.00 -> 52.0 mm, vias 0 -> 2
- net Net-(U6-GPIO0): track 0.00 -> 47.8 mm
- net Net-(U6-CHIP_PU): track 0.00 -> 43.3 mm, vias 0 -> 2
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- added copper zone on In2.Cu, net +3V3
- added copper zone on In1.Cu, net GND
Other:
- copper layers 2 -> 4

Commit message: upload
Parts:
- added G12312: LOGO, aslib:nl2, B.Cu at (104.0, 102.5)
- added G12321: LOGO, aslib:tux, F.Cu at (95.5, 39.5)
- added G12421: LOGO, aslib:hc_flag, F.Cu at (103.0, 113.5)
- added G21312: LOGO, aslib:github, B.Cu at (105.0, 161.5)
- added REF**: MountingHole_2.7mm_M2.5, MountingHole:MountingHole_2.7mm_M2.5, F.Cu at (133.5, 186.0)
- added REF**: MountingHole_2.7mm_M2.5, MountingHole:MountingHole_2.7mm_M2.5, F.Cu at (74.5, 186.0)
- moved J6 4.00 mm to (86.0, 186.0)
- moved R4 4.00 mm to (84.0, 177.5)
- moved R5 4.00 mm to (88.0, 177.5)
- moved R6 4.00 mm to (85.5, 179.5)
- moved R7 4.00 mm to (86.5, 179.5)
- moved U2 4.00 mm to (86.0, 177.0)
Connections:
- U6 pad 10: unconnected-(U6-GPIO5-Pad10) -> /COPROC_IRQ
Routing:
- net /MAIN_SDA: track 2.07 -> 296.9 mm, vias 0 -> 14
- net /MAIN_SCL: track 6.10 -> 287.4 mm, vias 0 -> 17
- net /SHIELD_DETECT: track 2.57 -> 181.2 mm, vias 0 -> 4
- net /MAIN_MOSI: track 154.0 -> 329.8 mm, vias 2 -> 14
- net /MAIN_SCLK: track 153.0 -> 325.1 mm, vias 5 -> 15
- net /COPROC_CS: track 0.00 -> 166.4 mm, vias 0 -> 4
- net /GPIO2: track 0.00 -> 153.1 mm, vias 0 -> 7
- net /COPROC_IRQ: track 0.00 -> 143.8 mm, vias 0 -> 4
- net /MAIN_MISO: track 154.6 -> 295.2 mm, vias 2 -> 15
- net /MOD0_CS: track 0.00 -> 126.1 mm, vias 0 -> 6
- net /MCU_DP: track 0.00 -> 118.3 mm, vias 0 -> 4
- net /MCU_DM: track 0.00 -> 118.0 mm, vias 0 -> 4
- net /IRQ2: track 0.00 -> 117.4 mm, vias 0 -> 2
- net /MOD1_CS: track 0.00 -> 110.8 mm, vias 0 -> 6
- net /NRF2_CS: track 0.00 -> 85.0 mm, vias 0 -> 4
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- added copper zone on B.Cu, net GND
- added copper zone on F.Cu, net GND
Other:
- board text added: "this board runs linux!"
