File: axiom_shield/axiom_shield.kicad_sch (KiCad schematic)
At the start: 2 parts, among them J2 MAINBOARD

Commit message: upload
Parts:
- added J10: RF4, symbol Connector:Conn_Coaxial
- added J11: RF2, symbol Connector:Conn_Coaxial
- added J12: RF1, symbol Connector:Conn_Coaxial
- added J13: RF3, symbol Connector:Conn_Coaxial
- added J14: CC1101, symbol Connector:Conn_Coaxial
Connections:
- net +3V3: now also J2.19 (Pin_19), J2.20 (Pin_20)
- net CC1101/ANT_OUT: now also J14.1 (In)
- net GND: now also J10.2 (Ext), J11.2 (Ext), J12.2 (Ext), J13.2 (Ext), J14.2 (Ext)
- net rf_mod_0/ANT: now also J12.1 (In)
- net rf_mod_1/ANT: now also J11.1 (In)
- net rf_mod_2/ANT: now also J13.1 (In)
- net rf_mod_3/ANT: now also J10.1 (In)
- no-connect marks 5 -> 3

Commit message: upload
Parts:
- J1: renamed from J12; footprint (none) -> Connector_Coaxial:SMA_Amphenol_901-144_Vertical
- J2: renamed from J13; footprint (none) -> Connector_Coaxial:SMA_Amphenol_901-144_Vertical
- J3: renamed from J11; footprint (none) -> Connector_Coaxial:SMA_Amphenol_901-144_Vertical
- J4: renamed from J10; footprint (none) -> Connector_Coaxial:SMA_Amphenol_901-144_Vertical
- J5: renamed from J2; footprint (none) -> Connector_PinSocket_2.54mm:PinSocket_2x10_P2.54mm_Vertical
- J6: renamed from J14; value CC1101 -> SUBGHZ; footprint (none) -> Connector_Coaxial:SMA_Amphenol_901-144_Vertical
- R1: renamed from R5; footprint (none) -> Resistor_SMD:R_0402_1005Metric
