File: axiom_shield/base_module.kicad_sch (KiCad schematic)
At the start: 1 part, among them J4 DF40C-20DP-0.4V_51_

Commit message: upload
Parts:
- removed J4: DF40C-20DP-0.4V_51_, DF40C-20DP-0.4V_51_:HRS_DF40C-20DP-0.4V_51_, symbol DF40C-20DP-0.4V_51_:DF40C-20DP-0.4V_51_
- added J10: DF40C-20DP-0.4V_51_, DF40C-20DP-0.4V_51_:HRS_DF40C-20DP-0.4V_51_, symbol DF40C-20DP-0.4V_51_:DF40C-20DP-0.4V_51_
Connections:
- net +3V3: now also J10.3, J10.4
- net +5V: now also J10.5, J10.6
- net GND: now also J10.1, J10.17, J10.18, J10.2, J10.7, J10.8
- net GPIO: now also J10.16
- net IRQ: now also J10.15
- net MOD_SCL: now also J10.14
- net MOD_SDA: now also J10.13
- net SPI_CS: now also J10.12
- net SPI_MISO: now also J10.10
- net SPI_MOSI: now also J10.9
- net SPI_SCK: now also J10.11
