File: axiom_shield/cc1101.kicad_sch (KiCad schematic)
At the start: 16 parts, among them U4 CC1101RGPR, Y2 XTM20026000FT00351005

Commit message: upload
Parts:
- C13: renamed from C12; footprint (none) -> Capacitor_SMD:C_0402_1005Metric
- C14: renamed from C11; footprint (none) -> Capacitor_SMD:C_0402_1005Metric
- C15: renamed from C10; footprint (none) -> Capacitor_SMD:C_0402_1005Metric
- C16: renamed from C9; footprint (none) -> Capacitor_SMD:C_0402_1005Metric
- C17: renamed from C13; footprint (none) -> Capacitor_SMD:C_0402_1005Metric
- C18: renamed from C14; value C_Small -> 100nF; footprint (none) -> Capacitor_SMD:C_0402_1005Metric
- C19: renamed from C15; footprint (none) -> Capacitor_SMD:C_0402_1005Metric
- C20: renamed from C16; footprint (none) -> Capacitor_SMD:C_0402_1005Metric
- C21: renamed from C17; footprint (none) -> Capacitor_SMD:C_0402_1005Metric
- C22: renamed from C18; footprint (none) -> Capacitor_SMD:C_0402_1005Metric
- C23: renamed from C19; footprint (none) -> Capacitor_SMD:C_0402_1005Metric
- L2: renamed from L1; footprint (none) -> Inductor_SMD:L_0402_1005Metric
- L3: renamed from L2; footprint (none) -> Inductor_SMD:L_0402_1005Metric
- R12: renamed from R8; footprint (none) -> Resistor_SMD:R_0402_1005Metric
- U6: renamed from U4; footprint CC1101RGPR:QFN50P400X400X100-21N -> misclib:cc1101
- Y2: footprint (none) -> Crystal:Crystal_SMD_2016-4Pin_2.0x1.6mm
Changed lines of the file:
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@@
 		(on_board yes)
 		(dnp no)
-		(property "Reference" "C17"
+		(property "Reference" "C21"
 			(at 211.836 93.98 0)
 			(effects
@@
 			)
 		)
-		(property "Footprint" ""
+		(property "Footprint" "Capacitor_SMD:C_0402_1005Metric"
 			(at 212.09 100.33 0)
 			(effects
@@
 			(project "axiom_shield"
 				(path "/17b1b55e-6df3-4e0d-982d-4199f16696cd/dfb6482e-9249-491f-a890-6eae73830776"
-					(reference "C17")
+					(reference "C21")
 					(unit 1)
 				)
@@
 		(on_board yes)
 		(dnp no)
-		(property "Reference" "C12"
+		(property "Reference" "C13"
 			(at 80.772 77.47 0)
 			(effects
@@
 			)
 		)
-		(property "Footprint" ""
+		(property "Footprint" "Capacitor_SMD:C_0402_1005Metric"
 			(at 88.9 81.28 0)
 			(effects
@@
 			(project "axiom_shield"
 				(path "/17b1b55e-6df3-4e0d-982d-4199f16696cd/dfb6482e-9249-491f-a890-6eae73830776"
-					(reference "C12")
+					(reference "C13")
 					(unit 1)
 				)
@@
 		(dnp no)
 		(fields_autoplaced yes)
-		(property "Reference" "#PWR022"
+		(property "Reference" "#PWR032"
 			(at 87.63 82.55 0)
 			(effects
@@
 			(project ""
 				(path "/17b1b55e-6df3-4e0d-982d-4199f16696cd/dfb6482e-9249-491f-a890-6eae73830776"
-					(reference "#PWR022")
+					(reference "#PWR032")
 					(unit 1)
 				)
@@
 		(on_board yes)
 		(dnp no)
-		(property "Reference" "C10"
+		(property "Reference" "C15"
 			(at 80.772 86.614 0)
 			(effects
@@
 			)
 		)
-		(property "Footprint" ""
+		(property "Footprint" "Capacitor_SMD:C_0402_1005Metric"
 			(at 93.98 86.36 0)
 			(effects
@@
 			(project "axiom_shield"
 				(path "/17b1b55e-6df3-4e0d-982d-4199f16696cd/dfb6482e-9249-491f-a890-6eae73830776"
-					(reference "C10")
+					(reference "C15")
 					(unit 1)
 				)
@@
 		(on_board yes)
 		(dnp no)
-		(property "Reference" "C19"
+		(property "Reference" "C23"
 			(at 236.22 93.98 0)
 			(effects
@@
 			)
 		)
-		(property "Footprint" ""
+		(property "Footprint" "Capacitor_SMD:C_0402_1005Metric"
 			(at 237.49 100.33 0)
 			(effects
@@
 			(project "axiom_shield"
 				(path "/17b1b55e-6df3-4e0d-982d-4199f16696cd/dfb6482e-9249-491f-a890-6eae73830776"
-					(reference "C19")
+					(reference "C23")
 					(unit 1)
 				)
@@
 		(dnp no)
 		(fields_autoplaced yes)
-		(property "Reference" "L2"
+		(property "Reference" "L3"
 			(at 187.96 99.06 90)
 			(effects
@@
 			)
 		)
-		(property "Footprint" ""
+		(property "Footprint" "Inductor_SMD:L_0402_1005Metric"
 			(at 187.96 104.14 0)
 			(effects
@@
 			(project "axiom_shield"
 				(path "/17b1b55e-6df3-4e0d-982d-4199f16696cd/dfb6482e-9249-491f-a890-6eae73830776"
-					(reference "L2")
+					(reference "L3")
 					(unit 1)
 				)
@@
 		(on_board yes)
 		(dnp no)
-		(property "Reference" "C18"
+		(property "Reference" "C22"
 			(at 219.456 100.33 0)
 			(effects
@@
 			)
 		)
-		(property "Footprint" ""
+		(property "Footprint" "Capacitor_SMD:C_0402_1005Metric"
 			(at 219.71 106.68 0)
 			(effects
@@
 			(project "axiom_shield"
 				(path "/17b1b55e-6df3-4e0d-982d-4199f16696cd/dfb6482e-9249-491f-a890-6eae73830776"
-					(reference "C18")
+					(reference "C22")
 					(unit 1)
 				)
@@
 		(dnp no)
 		(fields_autoplaced yes)
-		(property "Reference" "#PWR020"
+		(property "Reference" "#PWR033"
 			(at 109.22 100.33 0)
 			(effects
@@
 			(project "axiom_shield"
 				(path "/17b1b55e-6df3-4e0d-982d-4199f16696cd/dfb6482e-9249-491f-a890-6eae73830776"
-					(reference "#PWR020")
+					(reference "#PWR033")
 					(unit 1)
 				)
@@
 		(dnp no)
 		(fields_autoplaced yes)
-		(property "Reference" "#PWR019"
+		(property "Reference" "#PWR035"
 			(at 170.18 140.97 0)
 			(effects
@@
 			(project ""
 				(path "/17b1b55e-6df3-4e0d-982d-4199f16696cd/dfb6482e-9249-491f-a890-6eae73830776"
-					(reference "#PWR019")
+					(reference "#PWR035")
 					(unit 1)
 				)
@@
 		(on_board yes)
 		(dnp no)
-		(property "Reference" "C11"
+		(property "Reference" "C14"
 			(at 80.772 82.042 0)
 			(effects
@@
 			)
 		)
-		(property "Footprint" ""
+		(property "Footprint" "Capacitor_SMD:C_0402_1005Metric"
 			(at 91.44 83.82 0)
 			(effects
@@
 			(project "axiom_shield"
 				(path "/17b1b55e-6df3-4e0d-982d-4199f16696cd/dfb6482e-9249-491f-a890-6eae73830776"
-					(reference "C11")
+					(reference "C14")
 					(unit 1)
 				)
@@
 		(on_board yes)
 		(dnp no)
-		(property "Reference" "C16"
+		(property "Reference" "C20"
 			(at 182.626 107.442 0)
 			(effects
@@
 			)
 		)
-		(property "Footprint" ""
+		(property "Footprint" "Capacitor_SMD:C_0402_1005Metric"
 			(at 182.88 114.3 0)
 			(effects
@@
 			(project "axiom_shield"
 				(path "/17b1b55e-6df3-4e0d-982d-4199f16696cd/dfb6482e-9249-491f-a890-6eae73830776"
-					(reference "C16")
+					(reference "C20")
 					(unit 1)
 				)
@@
 		(on_board yes)
 		(dnp no)
-		(property "Reference" "C15"
+		(property "Reference" "C19"
 			(at 173.736 105.41 0)
 			(effects
@@
 			)
 		)
-		(property "Footprint" ""
+		(property "Footprint" "Capacitor_SMD:C_0402_1005Metric"
 			(at 173.99 111.76 0)
 			(effects
@@
 			(project ""
 				(path "/17b1b55e-6df3-4e0d-982d-4199f16696cd/dfb6482e-9249-491f-a890-6eae73830776"
-					(reference "C15")
+					(reference "C19")
 					(unit 1)
 				)
@@
 		(dnp no)
 		(fields_autoplaced yes)
-		(property "Reference" "U4"
+		(property "Reference" "U6"
 			(at 147.32 71.12 0)
 			(effects
@@
 			)
 		)
-		(property "Footprint" "CC1101RGPR:QFN50P400X400X100-21N"
+		(property "Footprint" "misclib:cc1101"
 			(at 147.32 106.68 0)
 			(effects
@@
 			(project ""
 				(path "/17b1b55e-6df3-4e0d-982d-4199f16696cd/dfb6482e-9249-491f-a890-6eae73830776"
-					(reference "U4")
+					(reference "U6")
 					(unit 1)
 				)
@@
 		(dnp no)
 		(fields_autoplaced yes)
-		(property "Reference" "L1"
+		(property "Reference" "L2"
 			(at 187.96 92.71 90)
 			(effects
@@
 			)
 		)
-		(property "Footprint" ""
+		(property "Footprint" "Inductor_SMD:L_0402_1005Metric"
 			(at 187.96 97.79 0)
 			(effects
@@
 			(project ""
 				(path "/17b1b55e-6df3-4e0d-982d-4199f16696cd/dfb6482e-9249-491f-a890-6eae73830776"
-					(reference "L1")
+					(reference "L2")
 					(unit 1)
 				)
@@
 		(dnp no)
 		(fields_autoplaced yes)
-		(property "Reference" "C14"
+		(property "Reference" "C18"
 			(at 121.9263 85.09 90)
 			(effects
@@
 			)
 		)
-		(property "Value" "C_Small"
+		(property "Value" "100nF"
 			(at 121.9263 87.63 90)
 			(effects
@@
 			)
 		)
-		(property "Footprint" ""
+		(property "Footprint" "Capacitor_SMD:C_0402_1005Metric"
 			(at 121.92 91.44 0)
 			(effects
@@
 			(project ""
 				(path "/17b1b55e-6df3-4e0d-982d-4199f16696cd/dfb6482e-9249-491f-a890-6eae73830776"
-					(reference "C14")
+					(reference "C18")
 					(unit 1)
 				)
@@
 		(dnp no)
 		(fields_autoplaced yes)
-		(property "Reference" "#PWR023"
+		(property "Reference" "#PWR036"
 			(at 219.71 115.57 0)
 			(effects
@@
 			(project "axiom_shield"
 				(path "/17b1b55e-6df3-4e0d-982d-4199f16696cd/dfb6482e-9249-491f-a890-6eae73830776"
-					(reference "#PWR023")
+					(reference "#PWR036")
 					(unit 1)
 				)
@@
 		(on_board yes)
 		(dnp no)
-		(property "Reference" "R8"
+		(property "Reference" "R12"
 			(at 121.92 124.206 90)
 			(effects
@@
 			)
 		)
-		(property "Footprint" ""
+		(property "Footprint" "Resistor_SMD:R_0402_1005Metric"
 			(at 121.92 121.92 0)
 			(effects
@@
 			(project ""
 				(path "/17b1b55e-6df3-4e0d-982d-4199f16696cd/dfb6482e-9249-491f-a890-6eae73830776"
-					(reference "R8")
+					(reference "R12")
 					(unit 1)
 				)
@@
 			)
 		)
-		(property "Footprint" ""
+		(property "Footprint" "Crystal:Crystal_SMD_2016-4Pin_2.0x1.6mm"
 			(at 199.39 113.03 0)
 			(effects
@@
 		(on_board yes)
 		(dnp no)
-		(property "Reference" "C9"
+		(property "Reference" "C16"
 			(at 80.772 91.694 0)
 			(effects
@@
 			)
 		)
-		(property "Footprint" ""
+		(property "Footprint" "Capacitor_SMD:C_0402_1005Metric"
 			(at 96.52 88.9 0)
 			(effects
@@
 			(project ""
 				(path "/17b1b55e-6df3-4e0d-982d-4199f16696cd/dfb6482e-9249-491f-a890-6eae73830776"
-					(reference "C9")
+					(reference "C16")
 					(unit 1)
 				)
@@
 		(on_board yes)
 		(dnp no)
-		(property "Reference" "C13"
+		(property "Reference" "C17"
 			(at 104.14 90.17 0)
 			(effects
@@
 			)
 		)
-		(property "Footprint" ""
+		(property "Footprint" "Capacitor_SMD:C_0402_1005Metric"
 			(at 101.6 91.44 0)
 			(effects
@@
 			(project "axiom_shield"
 				(path "/17b1b55e-6df3-4e0d-982d-4199f16696cd/dfb6482e-9249-491f-a890-6eae73830776"
-					(reference "C13")
+					(reference "C17")
 					(unit 1)
 				)
@@
 		(dnp no)
 		(fields_autoplaced yes)
-		(property "Reference" "#PWR021"
+		(property "Reference" "#PWR034"
 			(at 114.3 128.27 0)
 			(effects
@@
 			(project "axiom_shield"
 				(path "/17b1b55e-6df3-4e0d-982d-4199f16696cd/dfb6482e-9249-491f-a890-6eae73830776"
-					(reference "#PWR021")
-					(unit 1)
-				)
+					(reference "#PWR034")
+					(unit 1)
+				)
