File: axiom_shield/psu.kicad_sch (KiCad schematic)
At the start: 6 parts, among them J1 USB_C_Receptacle_USB2.0_14P, U1 USBLC6-2P6

Commit message: upload
Parts:
- added C21: 20uF, symbol Device:C
- added C22: 22uF, symbol Device:C
- added C23: 10uF, symbol Device:C
- added D1: LED1, symbol Device:LED
- added D2: LED2, symbol Device:LED
- added D3: LED3, symbol Device:LED
- added J9: BAT, symbol Connector_Generic:Conn_01x02
- added L3: 1uH, symbol Device:L
- added R10, R11, R12: 100, symbol Device:R
- added SW2: KEY, symbol Switch:SW_Push
- added U6: IP5306, IP5306:SOP127P600X165-9N, symbol IP5306:IP5306
Connections:
- net GND: now also C21.1, C22.2, C23.1, D1.1 (K), D2.1 (K), D3.1 (K), J9.2 (Pin_2), SW2.1, U6.9 (POWERPAD)
- net SHIELD_5V: now also C21.2, U6.8 (VOUT); no longer J1.A4 (VBUS), J1.A9 (VBUS), J1.B4 (VBUS), J1.B9 (VBUS)
- new net: D3.2 (A), R10.2
- new net: C22.1, J9.1 (Pin_1), L3.2, U6.6 (BAT)
- new net: D1.2 (A), R12.2
- new net: R10.1, U6.2 (LED1)
- new net: D2.2 (A), R11.2
- new net: SW2.2, U6.5 (KEY)
- new net: C23.2, J1.A4 (VBUS), J1.A9 (VBUS), J1.B4 (VBUS), J1.B9 (VBUS), U6.1 (VIN)
- new net: L3.1, U6.7 (SW)
- new net: R12.1, U6.4 (LED3)
- new net: R11.1, U6.3 (LED2)
Other:
- moved on the sheet: J1, R1, R2, R3, R4, U1

Commit message: upload
Parts:
- C10: renamed from C23; footprint (none) -> Capacitor_SMD:C_0402_1005Metric
- C11: renamed from C21; footprint (none) -> Capacitor_SMD:C_0402_1005Metric
- C12: renamed from C22; footprint (none) -> Capacitor_SMD:C_0402_1005Metric
- D1: renamed from D3; footprint (none) -> LED_SMD:LED_0603_1608Metric
- D2: footprint (none) -> LED_SMD:LED_0603_1608Metric
- D3: renamed from D1; footprint (none) -> LED_SMD:LED_0603_1608Metric
- J8: renamed from J1; footprint (none) -> Connector_USB:USB_C_Receptacle_HRO_TYPE-C-31-M-12
- J9: footprint (none) -> Connector_JST:JST_PH_B2B-PH-K_1x02_P2.00mm_Vertical
- L1: renamed from L3; footprint (none) -> Inductor_SMD:L_0402_1005Metric
- R10: renamed from R11; footprint (none) -> Resistor_SMD:R_0402_1005Metric
- R11: renamed from R12; footprint (none) -> Resistor_SMD:R_0402_1005Metric
- R5: renamed from R3; footprint (none) -> Resistor_SMD:R_0402_1005Metric
- R6: renamed from R4; footprint (none) -> Resistor_SMD:R_0402_1005Metric
- R7: renamed from R2; footprint (none) -> Resistor_SMD:R_0402_1005Metric
- R8: renamed from R1; footprint (none) -> Resistor_SMD:R_0402_1005Metric
- R9: renamed from R10; footprint (none) -> Resistor_SMD:R_0402_1005Metric
- SW2: footprint (none) -> Button_Switch_SMD:SW_SPST_B3U-1000P
- U5: renamed from U6; footprint IP5306:SOP127P600X165-9N -> misclib:ip5306
- renumbered U1 to U4
Changed lines of the file:
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@@
 		(on_board yes)
 		(dnp no)
-		(property "Reference" "R2"
+		(property "Reference" "R7"
 			(at 91.186 92.202 90)
 			(effects
@@
 			)
 		)
-		(property "Footprint" ""
+		(property "Footprint" "Resistor_SMD:R_0402_1005Metric"
 			(at 91.44 96.52 0)
 			(effects
@@
 			(project "axiom_shield"
 				(path "/17b1b55e-6df3-4e0d-982d-4199f16696cd/120cdb01-c78a-45e3-aaed-c9d7beac32f0"
-					(reference "R2")
+					(reference "R7")
 					(unit 1)
 				)
@@
 		(on_board yes)
 		(dnp no)
-		(property "Reference" "R3"
+		(property "Reference" "R5"
 			(at 74.676 83.058 90)
 			(effects
@@
 			)
 		)
-		(property "Footprint" ""
+		(property "Footprint" "Resistor_SMD:R_0402_1005Metric"
 			(at 74.93 86.36 0)
 			(effects
@@
 			(project "axiom_shield"
 				(path "/17b1b55e-6df3-4e0d-982d-4199f16696cd/120cdb01-c78a-45e3-aaed-c9d7beac32f0"
-					(reference "R3")
+					(reference "R5")
 					(unit 1)
 				)
@@
 		(on_board yes)
 		(dnp no)
-		(property "Reference" "D3"
+		(property "Reference" "D1"
 			(at 245.618 51.562 0)
 			(effects
@@
 			)
 		)
-		(property "Footprint" ""
+		(property "Footprint" "LED_SMD:LED_0603_1608Metric"
 			(at 232.41 53.34 0)
 			(effects
@@
 			(project "axiom_shield"
 				(path "/17b1b55e-6df3-4e0d-982d-4199f16696cd/120cdb01-c78a-45e3-aaed-c9d7beac32f0"
-					(reference "D3")
+					(reference "D1")
 					(unit 1)
 				)
@@
 		(on_board yes)
 		(dnp no)
-		(property "Reference" "R4"
+		(property "Reference" "R6"
 			(at 74.93 90.678 90)
 			(effects
@@
 			)
 		)
-		(property "Footprint" ""
+		(property "Footprint" "Resistor_SMD:R_0402_1005Metric"
 			(at 74.93 88.9 0)
 			(effects
@@
 			(project "axiom_shield"
 				(path "/17b1b55e-6df3-4e0d-982d-4199f16696cd/120cdb01-c78a-45e3-aaed-c9d7beac32f0"
-					(reference "R4")
+					(reference "R6")
 					(unit 1)
 				)
@@
 		(dnp no)
 		(fields_autoplaced yes)
-		(property "Reference" "C21"
+		(property "Reference" "C11"
 			(at 196.85 48.2599 0)
 			(effects
@@
 			)
 		)
-		(property "Footprint" ""
+		(property "Footprint" "Capacitor_SMD:C_0402_1005Metric"
 			(at 194.0052 53.34 0)
 			(effects
@@
 			(project ""
 				(path "/17b1b55e-6df3-4e0d-982d-4199f16696cd/120cdb01-c78a-45e3-aaed-c9d7beac32f0"
-					(reference "C21")
+					(reference "C11")
 					(unit 1)
 				)
@@
 		(dnp no)
 		(fields_autoplaced yes)
-		(property "Reference" "C22"
+		(property "Reference" "C12"
 			(at 223.52 80.0099 0)
 			(effects
@@
 			)
 		)
-		(property "Footprint" ""
+		(property "Footprint" "Capacitor_SMD:C_0402_1005Metric"
 			(at 220.6752 85.09 0)
 			(effects
@@
 			(project "axiom_shield"
 				(path "/17b1b55e-6df3-4e0d-982d-4199f16696cd/120cdb01-c78a-45e3-aaed-c9d7beac32f0"
-					(reference "C22")
+					(reference "C12")
 					(unit 1)
 				)
@@
 		(on_board yes)
 		(dnp no)
-		(property "Reference" "D1"
+		(property "Reference" "D3"
 			(at 245.618 61.722 0)
 			(effects
@@
 			)
 		)
-		(property "Footprint" ""
+		(property "Footprint" "LED_SMD:LED_0603_1608Metric"
 			(at 232.41 63.5 0)
 			(effects
@@
 			(project ""
 				(path "/17b1b55e-6df3-4e0d-982d-4199f16696cd/120cdb01-c78a-45e3-aaed-c9d7beac32f0"
-					(reference "D1")
+					(reference "D3")
 					(unit 1)
 				)
@@
 		(on_board yes)
 		(dnp no)
-		(property "Reference" "R10"
+		(property "Reference" "R9"
 			(at 212.09 53.594 90)
 			(effects
@@
 			)
 		)
-		(property "Footprint" ""
+		(property "Footprint" "Resistor_SMD:R_0402_1005Metric"
 			(at 212.09 60.198 90)
 			(effects
@@
 			(project ""
 				(path "/17b1b55e-6df3-4e0d-982d-4199f16696cd/120cdb01-c78a-45e3-aaed-c9d7beac32f0"
-					(reference "R10")
+					(reference "R9")
 					(unit 1)
 				)
@@
 		(dnp no)
 		(fields_autoplaced yes)
-		(property "Reference" "#PWR03"
+		(property "Reference" "#PWR027"
 			(at 81.28 95.25 0)
 			(effects
@@
 			(project "axiom_shield"
 				(path "/17b1b55e-6df3-4e0d-982d-4199f16696cd/120cdb01-c78a-45e3-aaed-c9d7beac32f0"
-					(reference "#PWR03")
+					(reference "#PWR027")
 					(unit 1)
 				)
@@
 		(dnp no)
 		(fields_autoplaced yes)
-		(property "Reference" "#PWR066"
+		(property "Reference" "#PWR031"
 			(at 236.22 73.66 0)
 			(effects
@@
 			(project "axiom_shield"
 				(path "/17b1b55e-6df3-4e0d-982d-4199f16696cd/120cdb01-c78a-45e3-aaed-c9d7beac32f0"
-					(reference "#PWR066")
+					(reference "#PWR031")
 					(unit 1)
 				)
@@
 			)
 		)
-		(property "Footprint" ""
+		(property "Footprint" "LED_SMD:LED_0603_1608Metric"
 			(at 232.41 58.42 0)
 			(effects
@@
 			)
 		)
-		(property "Footprint" ""
+		(property "Footprint" "Button_Switch_SMD:SW_SPST_B3U-1000P"
 			(at 140.97 63.5 0)
 			(effects
@@
 		(on_board yes)
 		(dnp no)
-		(property "Reference" "R1"
+		(property "Reference" "R8"
 			(at 91.44 101.346 90)
 			(effects
@@
 			)
 		)
-		(property "Footprint" ""
+		(property "Footprint" "Resistor_SMD:R_0402_1005Metric"
 			(at 91.44 99.06 0)
 			(effects
@@
 			(project ""
 				(path "/17b1b55e-6df3-4e0d-982d-4199f16696cd/120cdb01-c78a-45e3-aaed-c9d7beac32f0"
-					(reference "R1")
+					(reference "R8")
 					(unit 1)
 				)
@@
 			)
 		)
-		(property "Footprint" ""
+		(property "Footprint" "Connector_JST:JST_PH_B2B-PH-K_1x02_P2.00mm_Vertical"
 			(at 227.33 73.66 0)
 			(effects
@@
 		(dnp no)
 		(fields_autoplaced yes)
-		(property "Reference" "#PWR065"
+		(property "Reference" "#PWR030"
 			(at 208.28 87.63 0)
 			(effects
@@
 			(project ""
 				(path "/17b1b55e-6df3-4e0d-982d-4199f16696cd/120cdb01-c78a-45e3-aaed-c9d7beac32f0"
-					(reference "#PWR065")
+					(reference "#PWR030")
 					(unit 1)
 				)
@@
 		(dnp no)
 		(fields_autoplaced yes)
-		(property "Reference" "C23"
+		(property "Reference" "C10"
 			(at 149.86 48.2599 0)
 			(effects
@@
 			)
 		)
-		(property "Footprint" ""
+		(property "Footprint" "Capacitor_SMD:C_0402_1005Metric"
 			(at 147.0152 53.34 0)
 			(effects
@@
 			(project ""
 				(path "/17b1b55e-6df3-4e0d-982d-4199f16696cd/120cdb01-c78a-45e3-aaed-c9d7beac32f0"
-					(reference "C23")
+					(reference "C10")
 					(unit 1)
 				)
@@
 		(dnp no)
 		(fields_autoplaced yes)
-		(property "Reference" "U1"
+		(property "Reference" "U4"
 			(at 102.1781 88.9 0)
 			(effects
@@
 			(project ""
 				(path "/17b1b55e-6df3-4e0d-982d-4199f16696cd/120cdb01-c78a-45e3-aaed-c9d7beac32f0"
-					(reference "U1")
+					(reference "U4")
 					(unit 1)
 				)
@@
 		(dnp no)
 		(fields_autoplaced yes)
-		(property "Reference" "#PWR02"
+		(property "Reference" "#PWR028"
 			(at 99.06 110.49 0)
 			(effects
@@
 			(project "axiom_shield"
 				(path "/17b1b55e-6df3-4e0d-982d-4199f16696cd/120cdb01-c78a-45e3-aaed-c9d7beac32f0"
-					(reference "#PWR02")
+					(reference "#PWR028")
 					(unit 1)
 				)
@@
 		(dnp no)
 		(fields_autoplaced yes)
-		(property "Reference" "#PWR067"
+		(property "Reference" "#PWR029"
 			(at 146.05 76.2 0)
 			(effects
@@
 			(project "axiom_shield"
 				(path "/17b1b55e-6df3-4e0d-982d-4199f16696cd/120cdb01-c78a-45e3-aaed-c9d7beac32f0"
-					(reference "#PWR067")
+					(reference "#PWR029")
 					(unit 1)
 				)
@@
 		(dnp no)
 		(fields_autoplaced yes)
-		(property "Reference" "J1"
+		(property "Reference" "J8"
 			(at 57.15 73.66 0)
 			(effects
@@
 			)
 		)
-		(property "Footprint" ""
+		(property "Footprint" "Connector_USB:USB_C_Receptacle_HRO_TYPE-C-31-M-12"
 			(at 60.96 96.52 0)
 			(effects
@@
 			(project ""
 				(path "/17b1b55e-6df3-4e0d-982d-4199f16696cd/120cdb01-c78a-45e3-aaed-c9d7beac32f0"
-					(reference "J1")
+					(reference "J8")
 					(unit 1)
 				)
@@
 		(dnp no)
 		(fields_autoplaced yes)
-		(property "Reference" "L3"
+		(property "Reference" "L1"
 			(at 194.31 63.5 90)
 			(effects
@@
 			)
 		)
-		(property "Footprint" ""
+		(property "Footprint" "Inductor_SMD:L_0402_1005Metric"
 			(at 194.31 68.58 0)
 			(effects
@@
 			(project ""
 				(path "/17b1b55e-6df3-4e0d-982d-4199f16696cd/120cdb01-c78a-45e3-aaed-c9d7beac32f0"
-					(reference "L3")
+					(reference "L1")
 					(unit 1)
 				)
@@
 		(on_board yes)
 		(dnp no)
-		(property "Reference" "R12"
+		(property "Reference" "R11"
 			(at 212.09 58.674 90)
 			(effects
@@
 			)
 		)
-		(property "Footprint" ""
+		(property "Footprint" "Resistor_SMD:R_0402_1005Metric"
 			(at 212.09 65.278 90)
 			(effects
@@
 			(project "axiom_shield"
 				(path "/17b1b55e-6df3-4e0d-982d-4199f16696cd/120cdb01-c78a-45e3-aaed-c9d7beac32f0"
-					(reference "R12")
+					(reference "R11")
 					(unit 1)
 				)
@@
 		(on_board yes)
 		(dnp no)
-		(property "Reference" "R11"
+		(property "Reference" "R10"
 			(at 212.09 56.134 90)
 			(effects
@@
 			)
 		)
-		(property "Footprint" ""
+		(property "Footprint" "Resistor_SMD:R_0402_1005Metric"
 			(at 212.09 62.738 90)
 			(effects
@@
 			(project "axiom_shield"
 				(path "/17b1b55e-6df3-4e0d-982d-4199f16696cd/120cdb01-c78a-45e3-aaed-c9d7beac32f0"
-					(reference "R11")
+					(reference "R10")
 					(unit 1)
 				)
@@
 		(dnp no)
 		(fields_autoplaced yes)
-		(property "Reference" "#PWR01"
+		(property "Reference" "#PWR026"
 			(at 53.34 125.73 0)
 			(effects
@@
 			(project ""
 				(path "/17b1b55e-6df3-4e0d-982d-4199f16696cd/120cdb01-c78a-45e3-aaed-c9d7beac32f0"
-					(reference "#PWR01")
+					(reference "#PWR026")
 					(unit 1)
 				)
@@
 		(dnp no)
 		(fields_autoplaced yes)
-		(property "Reference" "U6"
+		(property "Reference" "U5"
 			(at 172.72 45.72 0)
 			(effects
@@
 			)
 		)
-		(property "Footprint" "IP5306:SOP127P600X165-9N"
+		(property "Footprint" "misclib:ip5306"
 			(at 172.72 66.04 0)
 			(effects
@@
 			(project ""
 				(path "/17b1b55e-6df3-4e0d-982d-4199f16696cd/120cdb01-c78a-45e3-aaed-c9d7beac32f0"
-					(reference "U6")
-					(unit 1)
-				)
+					(reference "U5")
+					(unit 1)
+				)
