File: axiom_shield/rp2040.kicad_sch (KiCad schematic)
At the start: 19 parts, among them J3 Conn_01x03_Pin, SW1 SW_Push, U2 RP2040, U3 W25Q128JVSIQ, U5 PCA9557PW, Y1 NX3225SA-12MHz-STD-CSR-6

Commit message: upload
Parts:
- SW1: value SW_Push -> RST
Connections:
- no-connect marks 2 -> 6
Changed lines of the file:
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@@
+	)
+	(no_connect
+		(at 170.18 73.66)
+	)
+	(no_connect
+		(at 170.18 129.54)
+	)
+	(no_connect
+		(at 170.18 132.08)
 	)
 	(no_connect
@@
 	(no_connect
 		(at 248.92 105.41)
+	)
+	(no_connect
+		(at 170.18 134.62)
 	)
 	(wire
@@
 			)
 		)
-		(property "Value" "SW_Push"
+		(property "Value" "RST"
 			(at 198.12 133.3499 90)
 			(effects

Commit message: upload
Parts:
- C1: renamed from C6; footprint (none) -> Capacitor_SMD:C_0402_1005Metric
- C2: renamed from C5; footprint (none) -> Capacitor_SMD:C_0402_1005Metric
- C3: renamed from C7; footprint (none) -> Capacitor_SMD:C_0402_1005Metric
- C4: renamed from C8; footprint (none) -> Capacitor_SMD:C_0402_1005Metric
- C5: renamed from C2; footprint (none) -> Capacitor_SMD:C_0402_1005Metric
- C6: renamed from C1; footprint (none) -> Capacitor_SMD:C_0402_1005Metric
- C7: renamed from C3; footprint (none) -> Capacitor_SMD:C_0402_1005Metric
- C8: renamed from C4; footprint (none) -> Capacitor_SMD:C_0402_1005Metric
- C9: renamed from C20; footprint (none) -> Capacitor_SMD:C_0402_1005Metric
- FB1: footprint (none) -> Inductor_SMD:L_0402_1005Metric
- J7: renamed from J3; footprint (none) -> Connector_PinHeader_2.54mm:PinHeader_1x03_P2.54mm_Vertical
- R2: renamed from R6; footprint (none) -> Resistor_SMD:R_0402_1005Metric
- R3: renamed from R7; footprint (none) -> Resistor_SMD:R_0402_1005Metric
- R4: renamed from R9; footprint (none) -> Resistor_SMD:R_0402_1005Metric
- SW1: footprint (none) -> Button_Switch_SMD:SW_SPST_B3U-1000P
- Y1: footprint (none) -> Crystal:Crystal_SMD_3225-4Pin_3.2x2.5mm
- renumbered U3 to U1, U5 to U3
